File: kleinSDR.sch (KiCad schematic (older format))
At the start: 33 parts

Commit message: Changed MCU to STM32F407VGT6
Parts:
- removed C? (x16): 100nF, Capacitor_SMD:C_0402_1005Metric, symbol Device:C_Small
- removed C? (x5): 1uF, Capacitor_SMD:C_0603_1608Metric, symbol Device:C
- removed C? (x2): 2.2uF, Capacitor_SMD:C_0603_1608Metric, symbol Device:C
- removed J?: DFU Mode, symbol Connector_Generic:Conn_01x02
- removed L?: 47u, Inductor_SMD:L_0603_1608Metric, symbol Device:L_Small
- removed R? (x2): 10k, Resistor_SMD:R_0402_1005Metric, symbol Device:R_Small
- removed R? (x3): 22E, Resistor_SMD:R_0402_1005Metric, symbol Device:R_Small
- removed U?: STM32F767ZITx, Package_QFP:LQFP-144_20x20mm_P0.5mm, symbol MCU_ST_STM32F7:STM32F767ZITx
- added R? (x2): 22E, Resistors_SMD:R_0402, symbol device:R_Small
- added U?: STM32F407VGTx, LQFP100, symbol stm32:STM32F407VGTx
Connections:
- net labels added: USB_OTG_FS_DM, USB_OTG_FS_DP
- net labels removed: +3V3, BOOT0, NRST
- wire segments 181 -> 37
Other:
- note added: "USB Connector"
- note removed: "Boot Mode"
- note removed: "Open GND Flash\nClose VDD DFU"
- note removed: "USB"

Commit message: Add buttons, encoders, USB and power
Add buttons, encoders, USB and power
Parts:
- removed U?: STM32F407VGTx, LQFP100, symbol stm32:STM32F407VGTx
- added C1, C10, C11, C12, C13, C14, C15, C16, C17, C2, C24, C3, C4, C5, C6, C7, C8, C9, C? (x9): 100nF, Capacitors_SMD:C_0603, symbol Device:C_Small
- added C18, C19, C20, C21, C22, C23: 1nF, Capacitors_SMD:C_0603, symbol Device:C_Small
- added C? (x3): 4.7uF, Capacitors_SMD:C_0603, symbol Device:C_Small
- added C? (x2): 2.2uF, Capacitors_SMD:C_0603, symbol Device:C_Small
- added J2: Frequency Dial, Pin_Headers:Pin_Header_Straight_1x04_Pitch2.54mm, symbol Connector_Generic:Conn_01x04
- added J?: SWDP, Pin_Headers:Pin_Header_Straight_1x04_Pitch2.54mm, symbol Connector_Generic:Conn_01x04
- added J?: Boot0, symbol Connector_Generic:Conn_01x02
- added J?: UART, symbol Connector_Generic:Conn_01x03
- added L?: 47uH, symbol Device:L_Small
- added R?: 10K, Resistors_SMD:R_0603, symbol Device:R_Small
- added R?: 47E, Resistors_SMD:R_0603, symbol Device:R_Small
- added SW1: PE6, Buttons_Switches_THT:SW_PUSH_6mm_h4.3mm, symbol Switch:SW_Push
- added SW10: PC15, Buttons_Switches_THT:SW_PUSH_6mm_h4.3mm, symbol Switch:SW_Push
- added SW11: PE3, Buttons_Switches_THT:SW_PUSH_6mm_h4.3mm, symbol Switch:SW_Push
- added SW12: PE5, Buttons_Switches_THT:SW_PUSH_6mm_h4.3mm, symbol Switch:SW_Push
- added SW13: PB0, Buttons_Switches_THT:SW_PUSH_6mm_h4.3mm, symbol Switch:SW_Push
- added SW14: PB2, Buttons_Switches_THT:SW_PUSH_6mm_h4.3mm, symbol Switch:SW_Push
- added SW15: PC4, Buttons_Switches_THT:SW_PUSH_6mm_h4.3mm, symbol Switch:SW_Push
- added SW16: PC5, Buttons_Switches_THT:SW_PUSH_6mm_h4.3mm, symbol Switch:SW_Push
- added SW17: PC13, Buttons_Switches_THT:SW_PUSH_6mm_h4.3mm, symbol Switch:SW_Push
- added SW18: Volume, symbol Device:Rotary_Encoder
- added SW19: RF Gain, symbol Device:Rotary_Encoder
- added SW2: PB8, Buttons_Switches_THT:SW_PUSH_6mm_h4.3mm, symbol Switch:SW_Push
- added SW20: RIT, symbol Device:Rotary_Encoder
- added SW3: PE4, Buttons_Switches_THT:SW_PUSH_6mm_h4.3mm, symbol Switch:SW_Push
- added SW4: PC0, Buttons_Switches_THT:SW_PUSH_6mm_h4.3mm, symbol Switch:SW_Push
- added SW5: PC14, Buttons_Switches_THT:SW_PUSH_6mm_h4.3mm, symbol Switch:SW_Push
- added SW6: PB3, Buttons_Switches_THT:SW_PUSH_6mm_h4.3mm, symbol Switch:SW_Push
- added SW7: PC1, Buttons_Switches_THT:SW_PUSH_6mm_h4.3mm, symbol Switch:SW_Push
- added SW8: PD6, Buttons_Switches_THT:SW_PUSH_6mm_h4.3mm, symbol Switch:SW_Push
- added SW9: PE2, Buttons_Switches_THT:SW_PUSH_6mm_h4.3mm, symbol Switch:SW_Push
- added U1: STM32F407VGTx, Package_QFP:LQFP-100_14x14mm_P0.5mm, symbol MCU_ST_STM32F4:STM32F407VGTx
- J1: renamed from J?; footprint (none) -> Connector_USB:USB_Mini-B_Lumberg_2486_01_Horizontal
- R1, R2: renamed from R?; footprint Resistors_SMD:R_0402 -> Resistors_SMD:R_0603; symbol device:R_Small -> Device:R_Small
- gave numbers to parts that had none: 1
Connections:
- net labels added: +3.3V, +3.3VA, +3.3VADC, +5V, ButtonBndM, ButtonBndP, ButtonF1, ButtonF2, ButtonF3, ButtonF4, ButtonF5, ButtonG1, ButtonG2, ButtonG3, ButtonG4, ButtonM1, ButtonM2, ButtonM3, ButtonPwr, ButtonStpM, ButtonStpP, EncFreq1, EncFreq2, EncRF1, EncRF2, EncRIT1, EncRIT2, EncVol1, EncVol2, NRST, SWCLK, SWDIO, UART_RX, UART_TX
- wire segments 37 -> 340
- no-connect marks 0 -> 1
Other:
- note added: "Buttons"
- note added: "Ceramic \nLow ESR"
- note added: "Frequency Dial \nOptical Encoder"
- note added: "Rotary Encoders"
- note added: "SWDP & Debug \nConnectors"
- note added: "Vdd, Vbat Decoupling"
- note added: "Vdda, Vref Decoupling"

Commit message: Decided to go back to F7
Parts:
- removed U1: STM32F407VGTx, Package_QFP:LQFP-100_14x14mm_P0.5mm, symbol MCU_ST_STM32F4:STM32F407VGTx
- added C?: 100nF, Capacitors_SMD:C_0603, symbol Device:C_Small
- added J?: Conn_01x30, symbol Connector_Generic:Conn_01x30
- added L?: 47uH, symbol Device:L_Small
- added U? (x2): WM8731, Housings_SSOP:SSOP-28_5.3x10.2mm_Pitch0.65mm, symbol pkl_kleinSDR:WM8731
- added U?: STM32F767ZITx, Package_QFP:LQFP-144_20x20mm_P0.5mm, symbol MCU_ST_STM32F7:STM32F767ZITx
- added U?: FOX924B-16.000, kleinSDR:FOX924B-16.000, symbol pkl_kleinSDR:FOX924B-16.000
- added U?: HY28B, kleinSDR:HY28B, symbol pkl_kleinSDR:HY28B
- SW18, SW19, SW20: footprint (none) -> Rotary_Encoder:RotaryEncoder_Alps_EC12E_Vertical_H20mm
Connections:
- net labels added: ADC1, ADC2, ADC3, BAND0, BAND1, BAND2, DAC1, DEMOD_I_OUT, DEMOD_Q_OUT, EXCITER_I_IN, EXCITER_Q_IN, PADDLE_DAH, PADDLE_DIT, PTT_ON, PWR_BUTTON, PWR_DWN, SCL, SDA, UI_3V, UI_5V, UI_8V
- wire segments 340 -> 431
- no-connect marks 1 -> 7
Other:
- note added: "TO DO:\n1. Check all pin assignments\n2. Check HSE/clock design\n3. Design power circuit"

Commit message: Add buttons, encoders, DFU USB connector, decoupling caps
Parts:
- added C? (x6): 100nF, Capacitors_SMD:C_0603, symbol Device:C_Small
- added R?: 10K, Resistors_SMD:R_0603, symbol Device:R_Small
- SW1: value PE6 -> PG6
- SW10: value PC15 -> PG15
- SW17: value PC13 -> PG2
- SW4: value PC0 -> PG11
- SW5: value PC14 -> PF0
- SW8: value PD6 -> PA15
Connections:
- wire segments 431 -> 469
Other:
- note added: "TO DO:\n1. Check all pin assignments\n2. Check HSE/clock design\n3. Design power circuit\n4. Can I make Cap 1 & 2 4.7uF?"
- note removed: "TO DO:\n1. Check all pin assignments\n2. Check HSE/clock design\n3. Design power circuit"
- moved on the sheet: J1

Commit message: Add HY28B connection
Connections:
- net labels added: LCD_BL, LCD_CS, LCD_D0, LCD_D1, LCD_D10, LCD_D11, LCD_D12, LCD_D13, LCD_D14, LCD_D15, LCD_D16, LCD_D17, LCD_D2, LCD_D3, LCD_D4, LCD_D5, LCD_D6, LCD_D7, LCD_RD, LCD_RESET, LCD_RS, LCD_SDI, LCD_SDO, LCD_WR, TP_CS, TP_IRQ, TP_SCK, TP_SDI, TP_SDO
- wire segments 469 -> 500
- no-connect marks 7 -> 9
Other:
- note added: "HY28B Connector"
