File: kleinSDR.sch (KiCad schematic (older format))
At the start: 84 parts, among them J1 USB_B_Mini, J2 Frequency Dial, SW1 PG6, SW10 PG15, SW11 PE3, SW12 PE5, SW13 PB0, SW14 PB2, SW15 PC4, SW16 PC5, SW17 PG2, SW18 Volume, SW19 RF Gain, SW2 PB8, SW20 RIT, SW3 PE4, SW4 PG11, SW5 PF0, SW6 PB3, SW7 PC1, SW8 PA15, SW9 PE2, U2 USBLC6-2SC6

Commit message: TX/RX Audio CODEC
Parts:
- removed U?: WM8731, Housings_SSOP:SSOP-28_5.3x10.2mm_Pitch0.65mm, symbol pkl_kleinSDR:WM8731
- added C? (x7): 100nF, Capacitors_SMD:C_0603, symbol Device:C_Small
- added C? (x3): 10uF, Capacitors_SMD:C_0603, symbol Device:C_Small
- added C? (x2): 470nF, Capacitors_SMD:C_0603, symbol Device:C_Small
- added C? (x2): 1uF, Capacitors_SMD:C_0603, symbol Device:C_Small
- added C? (x2): 220pF, Capacitors_SMD:C_0603, symbol Device:C_Small
- added R? (x5): 100E, Resistors_SMD:R_0603, symbol Device:R_Small
- added R? (x2): 47E, Resistors_SMD:R_0603, symbol Device:R_Small
- added R? (x2): 1K, Resistors_SMD:R_0603, symbol Device:R_Small
- added U?: WM8731, Housings_SSOP:SSOP-28_5.3x10.2mm_Pitch0.65mm, symbol pkl_kleinSDR:WM8731
Connections:
- net labels added: AUDIO_IN_I, AUDIO_IN_Q, AUDIO_OUT_I, AUDIO_OUT_Q, I2C4_SCL, I2C4_SDA, SAI2_FS_B, SAI2_MCLK_B, SAI2_SCK_B, SAI2_SD_A, SAI2_SD_B, VDDA
- wire segments 500 -> 645
- no-connect marks 9 -> 21
Other:
- note added: "Analog RX/TX Audio CODEC"
- note added: "I/Q RX/TX Audio CODEC"

Commit message: Add analog audio codec circuit
Parts:
- added C? (x2): 220uF, symbol Device:CP_Small
- added C? (x6): 1nF, Capacitors_SMD:C_0603, symbol Device:C_Small
- added C? (x2): 100nF, Capacitors_SMD:C_0603, symbol Device:C_Small
- added C? (x3): 1uF, Capacitors_SMD:C_0603, symbol Device:C_Small
- added C?: 220pF, Capacitors_SMD:C_0603, symbol Device:C_Small
- added C?: 10uF, Capacitors_SMD:C_0603, symbol Device:C_Small
- added J?: Line Out, symbol Connector:AudioJack3_Ground
- added J?: MIC IN, symbol Connector:AudioJack3_Ground
- added J?: LINE IN, symbol Connector:AudioJack3_Ground
- added J?: Line Out, symbol Connector_Generic:Conn_01x02
- added Q?: BC857, Package_TO_SOT_SMD:SOT-23, symbol Transistor_BJT:BC857
- added R? (x6): 100E, Resistors_SMD:R_0603, symbol Device:R_Small
- added R? (x2): 47E, Resistors_SMD:R_0603, symbol Device:R_Small
- added R? (x2): 1K, Resistors_SMD:R_0603, symbol Device:R_Small
- added R? (x5): 4k7, Resistors_SMD:R_0603, symbol Device:R_Small
- added R?: 680E, Resistors_SMD:R_0603, symbol Device:R_Small
- added R?: 47K, Resistors_SMD:R_0603, symbol Device:R_Small
Connections:
- net labels added: I2C2_SCL, I2C2_SDA, MICBIAS, PTT, SAI1_FS_B, SAI1_MCLK_B, SAI1_SCK_B, SAI1_SD_A, SAI1_SD_B
- wire segments 645 -> 758
- no-connect marks 21 -> 17

Commit message: Connect 30pin board to board
Parts:
- added R? (x2): 47E, Resistors_SMD:R_0603, symbol Device:R_Small
- J?: value Conn_01x30 -> 30pin Board to Board
Connections:
- net labels added: I2C1_SCL, I2C1_SDA
- net labels removed: SCL, SDA
- wire segments 758 -> 771
Other:
- note added: "TO DO:\n1. Check all pin assignments\n2. Check HSE/clock design\n3. Design power circuit\n4. Can I make Cap 1 & 2 4.7uF?\n5. Do paddle dah and dit connections\n"
- note removed: "TO DO:\n1. Check all pin assignments\n2. Check HSE/clock design\n3. Design power circuit\n4. Can I make Cap 1 & 2 4.7uF?"
Changed lines of the file:
@@
 ButtonPwr
 Wire Wire Line
-	3600 5400 3675 5400
+	3100 5400 3675 5400
 $Comp
 L Device:Rotary_Encoder SW18
@@
 	2375 4475 2375 4525
 Text Notes 10325 10450 0    50   ~ 0
-TO DO:\n1. Check all pin assignments\n2. Check HSE/clock design\n3. Design power circuit\n4. Can I make Cap 1 & 2 4.7uF?
+TO DO:\n1. Check all pin assignments\n2. Check HSE/clock design\n3. Design power circuit\n4. Can I make Cap 1 & 2 4.7uF?\n5. Do paddle dah and dit connections\n
 $Comp
 L Connector_Generic:Conn_01x30 J?
@@
 P 15925 2375
 F 0 "J?" H 15900 725 50  0000 L CNN
-F 1 "Conn_01x30" H 15725 3900 50  0000 L CNN
+F 1 "30pin Board to Board" H 15150 3950 50  0000 L CNN
 F 2 "" H 15925 2375 50  0001 C CNN
 F 3 "~" H 15925 2375 50  0001 C CNN
@@
 	15125 3375 15725 3375
 Connection ~ 15125 3875
-Text Label 15650 3275 2    50   ~ 0
-SDA
-Text Label 15650 3175 2    50   ~ 0
-SCL
+Text Label 15075 3275 2    50   ~ 0
+I2C1_SDA
+Text Label 15075 3175 2    50   ~ 0
+I2C1_SCL
 NoConn ~ 15650 3075
 NoConn ~ 15650 2975
@@
 Text Label 3600 7800 2    50   ~ 0
 SAI1_FS_B
-Text Label 6150 5800 0    50   ~ 0
+Text Label 6150 9200 0    50   ~ 0
 SAI1_SD_A
 Text Label 3600 7700 2    50   ~ 0
@@
 Wire Wire Line
 	12625 6525 12025 6525
+Text Label 6150 4000 0    50   ~ 0
+DAC1
+Wire Wire Line
+	6150 4000 6075 4000
+Text Label 3600 7200 2    50   ~ 0
+ADC3
+Wire Wire Line
+	3600 7200 3675 7200
+Text Label 6150 3800 0    50   ~ 0
+ADC2
+Wire Wire Line
+	6150 3800 6075 3800
+Text Label 6150 4100 0    50   ~ 0
+ADC1
+Wire Wire Line
+	6150 4100 6075 4100
+Text Label 6150 5300 0    50   ~ 0
+PTT_ON
+Wire Wire Line
+	6150 5300 6075 5300
+Text Label 6150 7700 0    50   ~ 0
+PWR_DWN
+Wire Wire Line
+	6150 7700 6075 7700
+Text Label 3600 5200 2    50   ~ 0
+BAND0
+Wire Wire Line
+	3600 5200 3675 5200
+Text Label 6150 4300 0    50   ~ 0
+BAND1
+Wire Wire Line
+	6150 4300 6075 4300
+Text Label 6150 4500 0    50   ~ 0
+BAND2
+Wire Wire Line
+	6150 4500 6075 4500
+Text Label 3100 5400 2    50   ~ 0
+PWR_BUTTON
+Wire Wire Line
+	6150 9200 6075 9200
+$Comp
+L Device:R_Small R?
+U 1 1 609D9B38
+P 15550 3175
+F 0 "R?" V 15525 3300 39  0000 C CNN
+F 1 "47E" V 15550 3175 39  0000 C CNN
+F 2 "Resistors_SMD:R_0603" H 15550 3175 50  0001 C CNN
+F 3 "~" H 15550 3175 50  0001 C CNN
+	1    15550 3175
+	0    1    1    0
+$EndComp
+$Comp
+L Device:R_Small R?
+U 1 1 609DA594
+P 15550 3275
+F 0 "R?" V 15525 3400 39  0000 C CNN
+F 1 "47E" V 15550 3275 39  0000 C CNN
+F 2 "Resistors_SMD:R_0603" H 15550 3275 50  0001 C CNN
+F 3 "~" H 15550 3275 50  0001 C CNN
+	1    15550 3275
+	0    1    1    0
+$EndComp
+Wire Wire Line
+	15450 3275 15075 3275
+Wire Wire Line
+	15450 3175 15075 3175
+Text Label 6150 5800 0    50   ~ 0
+I2C1_SCL
+Wire Wire Line
+	6075 5900 6150 5900
+Text Label 6150 5900 0    50   ~ 0
+I2C1_SDA
 $EndSCHEMATC

Commit message: Further updates
Parts:
- U3: renamed from U?; footprint Package_QFP:LQFP-144_20x20mm_P0.5mm -> Housings_QFP:LQFP-144_20x20mm_Pitch0.5mm
- gave numbers to parts that had none: 98

Commit message: Completed initial layout
Parts:
- removed C16, C46: 100nF, Capacitors_SMD:C_0603, symbol Device:C_Small
- removed C52: 10uF, Capacitors_SMD:C_0603, symbol Device:C_Small
- removed C64, C65: 220uF, symbol Device:CP_Small
- removed J6: Line Out, symbol Connector_Generic:Conn_01x02
- removed Q1: BC857, Package_TO_SOT_SMD:SOT-23, symbol Transistor_BJT:BC857
- removed R29, R30: 4k7, Resistors_SMD:R_0603, symbol Device:R_Small
- removed R31: 100E, Resistors_SMD:R_0603, symbol Device:R_Small
- removed SW1: PG6, Buttons_Switches_THT:SW_PUSH_6mm_h4.3mm, symbol Switch:SW_Push
- removed SW13: PB0, Buttons_Switches_THT:SW_PUSH_6mm_h4.3mm, symbol Switch:SW_Push
- removed SW14: PB2, Buttons_Switches_THT:SW_PUSH_6mm_h4.3mm, symbol Switch:SW_Push
- removed SW15: PC4, Buttons_Switches_THT:SW_PUSH_6mm_h4.3mm, symbol Switch:SW_Push
- removed SW16: PC5, Buttons_Switches_THT:SW_PUSH_6mm_h4.3mm, symbol Switch:SW_Push
- removed SW2: PB8, Buttons_Switches_THT:SW_PUSH_6mm_h4.3mm, symbol Switch:SW_Push
- removed SW3: PE4, Buttons_Switches_THT:SW_PUSH_6mm_h4.3mm, symbol Switch:SW_Push
- removed SW4: PG11, Buttons_Switches_THT:SW_PUSH_6mm_h4.3mm, symbol Switch:SW_Push
- removed SW5: PF0, Buttons_Switches_THT:SW_PUSH_6mm_h4.3mm, symbol Switch:SW_Push
- removed SW6: PB3, Buttons_Switches_THT:SW_PUSH_6mm_h4.3mm, symbol Switch:SW_Push
- removed SW7: PC1, Buttons_Switches_THT:SW_PUSH_6mm_h4.3mm, symbol Switch:SW_Push
- removed U3: STM32F767ZITx, Housings_QFP:LQFP-144_20x20mm_Pitch0.5mm, symbol MCU_ST_STM32F7:STM32F767ZITx
- removed U4: WM8731, Housings_SSOP:SSOP-28_5.3x10.2mm_Pitch0.65mm, symbol pkl_kleinSDR:WM8731
- added C16, C46: 220uF, symbol Device:CP_Small
- added C52: 10uF, symbol Device:CP_Small
- added C64: 470nF, Capacitors_SMD:C_0603, symbol Device:C_Small
- added C65: 220pF, Capacitors_SMD:C_0603, symbol Device:C_Small
- added C77, C78, C79: 1nF, Capacitors_SMD:C_0603, symbol Device:C_Small
- added J6: Line Out, symbol Connector:AudioJack3_Ground
- added L3: 47uH, symbol Device:L_Small
- added Q1: NDS356AP, symbol Device:Q_PMOS_DGS
- added U10: LM386, symbol Amplifier_Audio:LM386
- added U3, U4: 4066, symbol 4xxx:4066
- added U7: STM32F407VGTx, Package_QFP:LQFP-100_14x14mm_P0.5mm, symbol MCU_ST_STM32F4:STM32F407VGTx
- added U8, U9: MIC5504-3.3YM5, Package_TO_SOT_SMD:SOT-23-5, symbol Regulator_Linear:MIC5504-3.3YM5
- C1, C11, C12, C13, C2, C39, C40, C41, C42: value 100nF -> 1nF
- C27, C29: value 4.7uF -> 1uF
- C3: value 100nF -> 4.7uF
- C4, C43, C44, C48, C5, C55: value 100nF -> 1uF
- C45: value 4.7uF -> 220pF
- C47: value 100nF -> 47nF
- C49: value 10uF -> 100nF
- C50: value 470nF -> 10uF
- C51: value 470nF -> 100nF
- C53, C69: value 1uF -> 100nF
- C54: value 1uF -> 1nF
- C56: value 220pF -> 100nF
- C57, C71: value 220pF -> 470nF
- C6, C7: value 100nF -> 10uF
- C60, C62, C74: value 1nF -> 470nF
- C66: value 100nF -> 220pF
- C73, C75: value 1nF -> 1uF
- C76: value 1nF -> 100nF
- J7: value Line Out -> Phones
- J8: value LINE IN -> Microphone/PTT
- J9: value MIC IN -> Line In
- R10: value 100E -> 10E
- R11: value 47E -> 1K
- R12: value 47E -> 2K2
- R13, R14, R25: value 1K -> 4k7
- R20: value 680E -> 4k7
- R24: value 1K -> 4K7
- R26, R27: value 4k7 -> 4K7
- R28: value 47K -> 4K7
- R5: value 10K -> 2E2
- R6: value 100E -> 100
- R7: value 100E -> 47K
- R8: value 100E -> 0E
- R9: value 100E -> 2E2
Connections:
- net labels added: EN_IQIN, EN_LINEIN, I2S3_BCLK, I2S3_SD, I2S3_WS, I2S3_ext_SD, LINEIN_L, LINEIN_R, LINE_OUT, MIC_IN, RCC_MCO_2, Vref
- net labels removed: +3.3VADC, ButtonBndM, ButtonBndP, ButtonG1, ButtonG2, ButtonG3, ButtonG4, ButtonM1, ButtonM2, ButtonM3, ButtonStpM, ButtonStpP, I2C4_SCL, I2C4_SDA, MICBIAS, PTT, SAI1_FS_B, SAI1_MCLK_B, SAI1_SCK_B, SAI1_SD_A, SAI1_SD_B, SAI2_FS_B, SAI2_MCLK_B, SAI2_SCK_B, SAI2_SD_A, SAI2_SD_B, VDDA
- wire segments 771 -> 720
- no-connect marks 17 -> 18
Other:
- note added: "CODEC"
- note added: "Power"
- note removed: "Analog RX/TX Audio CODEC"
- note removed: "I/Q RX/TX Audio CODEC"

Commit message: Review/checked pin assignments, clock design, power circuits
Parts:
- removed C63: 10uF, Capacitors_SMD:C_0603, symbol Device:C_Small
- removed L1: 47uH, symbol Device:L_Small
- added C? (x2): 10uF, symbol Device:CP_Small
- added C?: 220uF, symbol Device:CP_Small
- added C?: 220pF, Capacitors_SMD:C_0603, symbol Device:C_Small
- added J?: 5V, symbol Connector_Generic:Conn_01x02
- added R?: 680, Resistors_SMD:R_0603, symbol Device:R_Small
- added R?: 4E7, Resistors_SMD:R_0603, symbol Device:R_Small
Connections:
- net labels added: MICBIAS
- wire segments 720 -> 739
- no-connect marks 18 -> 17
Other:
- note added: "Placed \nclosed \nto CPU"
- note added: "TO DO:\n1. Check all pin assignments - DONE\n2. Check HSE/clock design - DONE\n3. Design power circuit - DONE\n4. Can I make Cap 1 & 2 4.7uF?\n5. Do paddle dah and dit connections - DONE\n6. 0603 or 0402?\n7. MOSFET footprint\n8. Other footprints\n9. Check all decoupling caps\n"
- note added: "TODO: Add option to use VBUS"
- note removed: "TO DO:\n1. Check all pin assignments\n2. Check HSE/clock design\n3. Design power circuit\n4. Can I make Cap 1 & 2 4.7uF?\n5. Do paddle dah and dit connections\n"
- moved on the sheet: J1
